Commit message: Completed barista robot links and joints

File: urdf/barista_robot_model.urdf (robot description, URDF)
Before this commit: robot barista_robot, 4 links, 3 joints
Links:
- added link back_left_rod, mass 0.5; collision cylinder length=0.220 radius=0.01; visual cylinder length=0.220 radius=0.01
- added link back_pitch_link; visual sphere radius=0.0352
- added link back_right_rod, mass 0.5; collision cylinder length=0.220 radius=0.01; visual cylinder length=0.220 radius=0.01
- added link back_roll_link; visual cylinder length=0.05 radius=0.0152
- added link back_yaw_link; visual cylinder length=0.05 radius=0.0152
- added link cup_holder, mass 0.5; collision cylinder length=0.090 radius=0.160; visual cylinder length=0.090 radius=0.160
- added link front_left_rod, mass 0.5; collision cylinder length=0.220 radius=0.01; visual cylinder length=0.220 radius=0.01
- added link front_pitch_link; visual sphere radius=0.0352
- added link front_right_rod, mass 0.5; collision cylinder length=0.220 radius=0.01; visual cylinder length=0.220 radius=0.01
- added link front_roll_link; visual cylinder length=0.05 radius=0.0152
- added link front_yaw_link; visual cylinder length=0.05 radius=0.0152
Joints:
- added joint back_left_rod_joint: type continuous, parent chassis, child back_left_rod, origin xyz=-0.090 0.090 0.0775 rpy=0 0 0, axis 0 0 1, limit effort=10000 velocity=1000
- added joint back_pitch_joint: type continuous, parent back_roll_link, child back_pitch_link, origin xyz=0 0 0 rpy=0 0 0, axis 0 1 0, limit effort=1000.0 velocity=100.0
- added joint back_right_rod_joint: type continuous, parent chassis, child back_right_rod, origin xyz=-0.090 -0.090 0.0775 rpy=0 0 0, axis 0 0 1, limit effort=10000 velocity=1000
- added joint back_roll_joint: type continuous, parent back_yaw_link, child back_roll_link, origin xyz=0 0 0 rpy=0 0 0, axis 1 0 0, limit effort=1000.0 velocity=100.0
- added joint back_yaw_joint: type continuous, parent chassis, child back_yaw_link, origin xyz=-0.128 0 -0.075 rpy=0 0 0, axis 0 0 1, limit effort=1000.0 velocity=100.0
- added joint cup_holder_joint: type continuous, parent chassis, child cup_holder, origin xyz=0 0 0.3425 rpy=0 0 0, axis 0 0 1, limit effort=10000 velocity=1000
- added joint front_left_rod_joint: type continuous, parent chassis, child front_left_rod, origin xyz=0.090 0.090 0.0775 rpy=0 0 0, axis 0 0 1, limit effort=10000 velocity=1000
- added joint front_pitch_joint: type continuous, parent front_roll_link, child front_pitch_link, origin xyz=0 0 0 rpy=0 0 0, axis 0 1 0, limit effort=1000.0 velocity=100.0
- added joint front_right_rod_joint: type continuous, parent chassis, child front_right_rod, origin xyz=0.090 -0.090 0.0775 rpy=0 0 0, axis 0 0 1, limit effort=10000 velocity=1000
- added joint front_roll_joint: type continuous, parent front_yaw_link, child front_roll_link, origin xyz=0 0 0 rpy=0 0 0, axis 1 0 0, limit effort=1000.0 velocity=100.0
- added joint front_yaw_joint: type continuous, parent chassis, child front_yaw_link, origin xyz=0.128 0 -0.075 rpy=0 0 0, axis 0 0 1, limit effort=1000.0 velocity=100.0

Commit message: Computed inertia for links

File: urdf/barista_robot_model.urdf (robot description, URDF)
Before this commit: robot barista_robot, 15 links, 14 joints
Links:
- link back_left_rod: mass 0.5 -> 0.250
- link back_pitch_link: mass None -> 0.1; geometry collision sphere radius=0.0352; visual sphere radius=0.0352
- link back_right_rod: mass 0.5 -> 0.250
- link chassis: mass 0.5 -> 2.5
- link cup_holder: mass 0.5 -> 1.0
- link front_left_rod: mass 0.5 -> 0.250
- link front_pitch_link: mass None -> 0.1; geometry collision sphere radius=0.0352; visual sphere radius=0.0352
- link front_right_rod: mass 0.5 -> 0.250
- link left_motor_wheel: mass 0.5 -> 0.1
- link right_motor_wheel: mass 0.5 -> 0.1

Commit message: Added a laser sensor to urdf model

File: urdf/barista_robot_model.urdf (robot description, URDF)
Before this commit: robot barista_robot, 15 links, 14 joints
Links:
- added link laser_scan_link, mass 0.01; collision box size=0.1 0.1 0.08; visual mesh filename=package://barista_robot_description/meshes/hokuyo_urg_04lx.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 scale=1.0 1.0 1.0
Joints:
- added joint laser_scan_link_joint: type fixed, parent chassis, child laser_scan_link, origin xyz=0.090 0 0.0775 rpy=0 0 0

Commit message: Corrected offset and collision on caster wheels

File: urdf/barista_robot_model.urdf (robot description, URDF)
Before this commit: robot barista_robot, 16 links, 15 joints
Links:
- link back_roll_link: mass None -> 0.1; geometry collision cylinder length=0.05 radius=0.0152; visual cylinder length=0.05 radius=0.0152
- link back_yaw_link: mass None -> 0.1; geometry collision cylinder length=0.05 radius=0.0152; visual cylinder length=0.05 radius=0.0152
- link front_roll_link: mass None -> 0.1; geometry collision cylinder length=0.05 radius=0.0152; visual cylinder length=0.05 radius=0.0152
- link front_yaw_link: mass None -> 0.1; geometry collision cylinder length=0.05 radius=0.0152; visual cylinder length=0.05 radius=0.0152
Joints:
- joint back_yaw_joint: origin xyz=-0.128 0 -0.075 rpy=0 0 0 -> xyz=-0.128 0 -0.0775 rpy=0 0 0
- joint front_yaw_joint: origin xyz=0.128 0 -0.075 rpy=0 0 0 -> xyz=0.128 0 -0.0775 rpy=0 0 0

Commit message: Corrected inertia values for caster wheels

File: urdf/barista_robot_model.urdf (robot description, URDF)
Before this commit: robot barista_robot, 16 links, 15 joints
Links:
- link front_roll_link: mass 0.1 -> 0.01
- link front_yaw_link: mass 0.1 -> 0.01
- link laser_scan_link: mass 0.01 -> 0.160

Commit message: Switched all joints parent link to base_link

File: urdf/barista_robot_model.urdf (robot description, URDF)
Before this commit: robot barista_robot, 16 links, 15 joints
Joints:
- joint back_left_rod_joint: origin xyz=-0.090 0.090 0.0775 rpy=0 0 0 -> xyz=-0.090 0.090 0.1902 rpy=0 0 0; parent chassis -> base_link
- joint back_right_rod_joint: origin xyz=-0.090 -0.090 0.0775 rpy=0 0 0 -> xyz=-0.090 -0.090 0.1902 rpy=0 0 0; parent chassis -> base_link
- joint back_yaw_joint: origin xyz=-0.128 0 -0.0775 rpy=0 0 0 -> xyz=-0.128 0 0.0352 rpy=0 0 0; parent chassis -> base_link
- joint cup_holder_joint: origin xyz=0 0 0.3425 rpy=0 0 0 -> xyz=0 0 0.4552 rpy=0 0 0; parent chassis -> base_link
- joint front_left_rod_joint: origin xyz=0.090 0.090 0.0775 rpy=0 0 0 -> xyz=0.090 0.090 0.1902 rpy=0 0 0; parent chassis -> base_link
- joint front_right_rod_joint: origin xyz=0.090 -0.090 0.0775 rpy=0 0 0 -> xyz=0.090 -0.090 0.1902 rpy=0 0 0; parent chassis -> base_link
- joint front_yaw_joint: origin xyz=0.128 0 -0.0775 rpy=0 0 0 -> xyz=0.128 0 0.0352 rpy=0 0 0; parent chassis -> base_link
- joint laser_scan_link_joint: origin xyz=0.090 0 0.0775 rpy=0 0 0 -> xyz=0.090 0 0.2302 rpy=0 0 0; parent chassis -> base_link
- joint left_motor_wheel_joint: origin xyz=0 0.158 -0.0775 rpy=0 0 0 -> xyz=0 0.158 0.0352 rpy=0 0 0; parent chassis -> base_link
- joint right_motor_wheel_joint: origin xyz=0 -0.158 -0.0775 rpy=0 0 0 -> xyz=0 -0.158 0.0352 rpy=0 0 0; parent chassis -> base_link

Commit message: Added Diff Drive plugin and adjusted rods positions

File: urdf/barista_robot_model.urdf (robot description, URDF)
Before this commit: robot barista_robot, 16 links, 15 joints
Joints:
- joint back_left_rod_joint: axis 0 0 1 -> (none); limit effort=10000 velocity=1000 -> (none); origin xyz=-0.090 0.090 0.1902 rpy=0 0 0 -> xyz=-0.020 0.130 0.1902 rpy=0 0 0; type continuous -> fixed
- joint back_right_rod_joint: axis 0 0 1 -> (none); limit effort=10000 velocity=1000 -> (none); origin xyz=-0.090 -0.090 0.1902 rpy=0 0 0 -> xyz=-0.020 -0.130 0.1902 rpy=0 0 0; type continuous -> fixed
- joint cup_holder_joint: axis 0 0 1 -> (none); limit effort=10000 velocity=1000 -> (none); type continuous -> fixed
- joint front_left_rod_joint: axis 0 0 1 -> (none); limit effort=10000 velocity=1000 -> (none); origin xyz=0.090 0.090 0.1902 rpy=0 0 0 -> xyz=0.050 0.130 0.1902 rpy=0 0 0; type continuous -> fixed
- joint front_right_rod_joint: axis 0 0 1 -> (none); limit effort=10000 velocity=1000 -> (none); origin xyz=0.090 -0.090 0.1902 rpy=0 0 0 -> xyz=0.050 -0.130 0.1902 rpy=0 0 0; type continuous -> fixed
- joint laser_scan_link_joint: origin xyz=0.090 0 0.2302 rpy=0 0 0 -> xyz=0.110 0 0.2302 rpy=0 0 0
