Commit message: Adjusted joint parameters

File: xacro/cup_holder_tray.xacro (robot description, xacro)
@@ -30,7 +30,4 @@
             <parent link="${parent}" />
             <child link="${child}" />
-            <axis rpy="0 0 0" xyz="0 0 1"/>
-            <limit effort="10000" velocity="1000"/>
-            <joint_properties damping="1.0" friction="1.0"/>
         </joint>
     </xacro:macro>

File: xacro/standoff_rod.xacro (robot description, xacro)
@@ -30,7 +30,4 @@
             <parent link="${parent}" />
             <child link="${child}" />
-            <axis rpy="0 0 0" xyz="0 0 1"/>
-            <limit effort="10000" velocity="1000"/>
-            <joint_properties damping="1.0" friction="1.0"/>
         </joint>
     </xacro:macro>
