Commit message: Added standoff rods macro to robot model

File: xacro/barista_robot_model.urdf.xacro (robot description, xacro)
@@ -5,4 +5,6 @@
     <!--Include caster wheels macros -->
     <xacro:include filename="$(find barista_robot_description)/xacro/caster_wheel.xacro"/>
+    <!--Include standoff rods macros -->
+    <xacro:include filename="$(find barista_robot_description)/xacro/standoff_rod.xacro"/>
     <material name="red">
       <color rgba="1.0 0.0 0.0 1"/>
@@ -23,4 +25,5 @@
         <color rgba="0.0 0.0 1.0 1"/>
     </material>
+    <!--Base Link-->
     <link name="base_link"></link>
     <!-- Body -->
@@ -41,5 +44,6 @@
             <mass value="2.5"/>
             <origin rpy="0 0 0" xyz="0 0 0"/>
-            <inertia ixx="0.024807708333333334" ixy="0" ixz="0" iyy="0.024807708333333334" iyz="0" izz="0.039604999999999994"/>
+            <inertia ixx="0.024807708333333334" ixy="0" ixz="0"
+                iyy="0.024807708333333334" iyz="0" izz="0.039604999999999994"/>
         </inertial>
     </link>
@@ -49,4 +53,5 @@
         <child link="chassis" />
     </joint>
+    <!--******************** Drive Wheels **************************-->
     <!--Right drive wheel-->
     <xacro:drive_wheel wheel_name="right_motor_wheel" origin_xyz="0 0 0"
@@ -61,4 +66,5 @@
         origin_xyz="0 0.158 0.0352" origin_rpy="0 0 0" parent="base_link"
         child="left_motor_wheel" axis_xyz="0 1 0"/>
+    <!--******************** Caster Wheels **************************-->
     <!--Caster wheels are modeled by 3 different links for each representing one RPY angle-->
     <!--We use the drive_wheel macro to represent Yaw and Roll links-->
@@ -81,5 +87,4 @@
         origin_xyz="0 0 0" origin_rpy="0 0 0" parent="front_roll_link"
         child="front_pitch_link" axis_xyz="0 1 0"/>
-    <!--*************************************************************************************************-->
     <!-- Back Caster wheel Yaw Link and Joint-->
     <xacro:drive_wheel wheel_name="back_yaw_link" origin_xyz="0 0 0"
@@ -100,3 +105,30 @@
         origin_xyz="0 0 0" origin_rpy="0 0 0" parent="back_roll_link"
         child="back_pitch_link" axis_xyz="0 1 0"/>
+    <!--******************** Standoff Rods **************************-->
+    <!--Standoff Rods Links and joints-->
+    <!--Front Right Rod-->
+    <xacro:standoff_rod rod_name="front_right_rod" origin_xyz="0 0 0.110"
+            origin_rpy="0 0 0" r_l="0.220" r_r="0.01" material="white" mass="0.250"/>
+    <xacro:rod_joint joint_name="front_right_rod_joint" type="continuous"
+        origin_xyz="0.090 -0.090 0.1902" origin_rpy="0 0 0" parent="base_link"
+        child="front_right_rod"/>
+    <!--Front Left Rod-->
+    <xacro:standoff_rod rod_name="front_left_rod" origin_xyz="0 0 0.110"
+            origin_rpy="0 0 0" r_l="0.220" r_r="0.01" material="white" mass="0.250"/>
+    <xacro:rod_joint joint_name="front_left_rod_joint" type="continuous"
+        origin_xyz="0.090 0.090 0.1902" origin_rpy="0 0 0" parent="base_link"
+        child="front_left_rod"/>
+    <!--Back Right Rod-->
+    <xacro:standoff_rod rod_name="back_right_rod" origin_xyz="0 0 0.110"
+            origin_rpy="0 0 0" r_l="0.220" r_r="0.01" material="white" mass="0.250"/>
+    <xacro:rod_joint joint_name="back_right_rod_joint" type="continuous"
+        origin_xyz="-0.090 -0.090 0.1902" origin_rpy="0 0 0" parent="base_link"
+        child="back_right_rod"/>
+    <!--Back Left Rod-->
+    <xacro:standoff_rod rod_name="back_left_rod" origin_xyz="0 0 0.110"
+            origin_rpy="0 0 0" r_l="0.220" r_r="0.01" material="white" mass="0.250"/>
+    <xacro:rod_joint joint_name="back_left_rod_joint" type="continuous"
+        origin_xyz="-0.090 0.090 0.1902" origin_rpy="0 0 0" parent="base_link"
+        child="back_left_rod"/>
+    <!--******************** Cup Holder Tray **************************-->
 </robot>

Commit message: Added gazebo tags to xacro model for better visualization

File: xacro/barista_robot_model.urdf.xacro (robot description, xacro)
@@ -55,4 +55,7 @@
         <child link="chassis" />
     </joint>
+    <gazebo reference="chassis">
+        <material>Gazebo/Blue</material>
+    </gazebo>
     <!--******************** Drive Wheels **************************-->
     <!--Right drive wheel-->
@@ -62,4 +65,9 @@
         origin_xyz="0 -0.158 0.0352" origin_rpy="0 0 0" parent="base_link"
         child="right_motor_wheel" axis_xyz="0 1 0"/>
+    <gazebo reference="right_motor_wheel">
+        <mu1>0.7</mu1>
+        <mu2>0.7</mu2>
+        <material>Gazebo/Black</material>
+    </gazebo>
     <!--Left drive wheel-->
     <xacro:drive_wheel wheel_name="left_motor_wheel" origin_xyz="0 0 0"
@@ -68,4 +76,9 @@
         origin_xyz="0 0.158 0.0352" origin_rpy="0 0 0" parent="base_link"
         child="left_motor_wheel" axis_xyz="0 1 0"/>
+    <gazebo reference="left_motor_wheel">
+        <mu1>0.7</mu1>
+        <mu2>0.7</mu2>
+        <material>Gazebo/Black</material>
+    </gazebo>
     <!--******************** Caster Wheels **************************-->
     <!--Caster wheels are modeled by 3 different links for each representing one RPY angle-->
@@ -89,4 +102,9 @@
         origin_xyz="0 0 0" origin_rpy="0 0 0" parent="front_roll_link"
         child="front_pitch_link" axis_xyz="0 1 0"/>
+    <gazebo reference="front_pitch_link">
+        <mu1>0.0</mu1>
+        <mu2>0.0</mu2>
+        <material>Gazebo/Green</material>
+    </gazebo>
     <!-- Back Caster wheel Yaw Link and Joint-->
     <xacro:drive_wheel wheel_name="back_yaw_link" origin_xyz="0 0 0"
@@ -107,4 +125,9 @@
         origin_xyz="0 0 0" origin_rpy="0 0 0" parent="back_roll_link"
         child="back_pitch_link" axis_xyz="0 1 0"/>
+    <gazebo reference="back_pitch_link">
+        <mu1>0.0</mu1>
+        <mu2>0.0</mu2>
+        <material>Gazebo/Green</material>
+    </gazebo>
     <!--******************** Standoff Rods **************************-->
     <!--Standoff Rods Links and joints-->
@@ -115,4 +138,7 @@
         origin_xyz="0.090 -0.090 0.1902" origin_rpy="0 0 0" parent="base_link"
         child="front_right_rod"/>
+    <gazebo reference="front_right_rod">
+        <material>Gazebo/White</material>
+    </gazebo>
     <!--Front Left Rod-->
     <xacro:standoff_rod rod_name="front_left_rod" origin_xyz="0 0 0.110"
@@ -121,4 +147,7 @@
         origin_xyz="0.090 0.090 0.1902" origin_rpy="0 0 0" parent="base_link"
         child="front_left_rod"/>
+    <gazebo reference="front_left_rod">
+        <material>Gazebo/White</material>
+    </gazebo>
     <!--Back Right Rod-->
     <xacro:standoff_rod rod_name="back_right_rod" origin_xyz="0 0 0.110"
@@ -127,4 +156,7 @@
         origin_xyz="-0.090 -0.090 0.1902" origin_rpy="0 0 0" parent="base_link"
         child="back_right_rod"/>
+    <gazebo reference="back_right_rod">
+        <material>Gazebo/White</material>
+    </gazebo>
     <!--Back Left Rod-->
     <xacro:standoff_rod rod_name="back_left_rod" origin_xyz="0 0 0.110"
@@ -133,4 +165,7 @@
         origin_xyz="-0.090 0.090 0.1902" origin_rpy="0 0 0" parent="base_link"
         child="back_left_rod"/>
+    <gazebo reference="back_left_rod">
+        <material>Gazebo/White</material>
+    </gazebo>
     <!--******************** Cup Holder Tray **************************-->
     <xacro:cup_holder_tray link_name="cup_holder" origin_xyz="0 0 0"
@@ -139,3 +174,6 @@
         origin_xyz="0 0 0.4552" origin_rpy="0 0 0" parent="base_link"
         child="cup_holder"/>
+    <gazebo reference="cup_holder">
+        <material>Gazebo/Blue</material>
+    </gazebo>
 </robot>

Commit message: Added laser scan macro

File: xacro/barista_robot_model.urdf.xacro (robot description, xacro)
@@ -9,4 +9,6 @@
     <!--Include cup holder tray macro -->
     <xacro:include filename="$(find barista_robot_description)/xacro/cup_holder_tray.xacro"/>
+    <!--Include laser or not in representation-->
+    <xacro:property name="include_laser" value="true"/>
     <material name="red">
       <color rgba="1.0 0.0 0.0 1"/>
@@ -177,3 +179,73 @@
         <material>Gazebo/Blue</material>
     </gazebo>
+    <!--********************Laser Scan **************************-->
+    <xacro:macro name="laser" params="include_laser:=true">
+        <xacro:if value="${include_laser}">
+            <!-- Laser Sensor -->
+            <link name="laser_scan_link">
+                <visual>
+                    <origin rpy="0 0 0" xyz="0 0 -0.04"/>
+                    <geometry>
+                        <mesh filename="package://barista_robot_description/meshes/hokuyo_urg_04lx.dae" scale="1.0 1.0 1.0"/>
+                    </geometry>
+                </visual>
+                <collision>
+                    <origin rpy="0 0 0" xyz="0 0 0"/>
+                    <geometry>
+                        <box size="0.1 0.1 0.08"/>
+                    </geometry>
+                </collision>
+                <inertial>
+                    <mass value="0.160"/>
+                    <origin rpy="0 0 0" xyz="0 0 0"/>
+                    <inertia ixx="0.0002186666666666667" ixy="0" ixz="0" iyy="0.0002186666666666667" iyz="0" izz="0.00026666666666666673"/>
+                </inertial>
+            </link>
+            <joint name="laser_scan_link_joint" type="fixed">
+                <origin rpy="0 0 0" xyz="0.090 0 0.2302"/> <!--z = 0.0352 + 0.155 + 0.08/2-->
+                <parent link="base_link"/>
+                <child link="laser_scan_link"/>
+            </joint>
+            <gazebo reference="laser_scan_link">
+                <mu1>10.0</mu1>
+                <mu2>10.0</mu2>
+                <material>Gazebo/Grey</material>
+            </gazebo>
+            <gazebo reference="laser_scan_link">
+                <sensor name="sensor_ray" type="ray">
+                    <pose>0 0 0 0 0 0</pose>
+                    <ray>
+                        <scan>
+                            <horizontal>
+                                <samples>200</samples>
+                                <resolution>1.0</resolution>
+                                <min_angle>-1.5707</min_angle>
+                                <max_angle>1.5707</max_angle>
+                            </horizontal>
+                        </scan>
+                        <range>
+                            <min>0.2</min>
+                            <max>4.0</max>
+                        </range>
+                        <noise>
+                            <type>gaussian</type>
+                            <mean>0.0</mean>
+                            <stddev>0.01</stddev>
+                        </noise>
+                    </ray>
+                    <always_on>true</always_on>
+                    <visualize>true</visualize>
+                    <update_rate>100</update_rate>
+                    <plugin name="laser" filename="libgazebo_ros_ray_sensor.so">
+                        <ros>
+                            <!-- <namespace>/barista_robot</namespace> -->
+                            <remapping>~/out:=scan</remapping>
+                        </ros>
+                        <output_type>sensor_msgs/LaserScan</output_type>
+                    </plugin>
+                </sensor>
+            </gazebo>
+        </xacro:if>
+    </xacro:macro>
+    <xacro:laser include_laser="${include_laser}"/>
 </robot>

Commit message: Added laser_scan xacro file

File: xacro/barista_robot_model.urdf.xacro (robot description, xacro)
@@ -11,4 +11,5 @@
     <!--Include laser or not in representation-->
     <xacro:property name="include_laser" value="true"/>
+    <xacro:include filename="$(find barista_robot_description)/xacro/laser_scanner.xacro"/>
     <material name="red">
       <color rgba="1.0 0.0 0.0 1"/>
@@ -137,6 +138,6 @@
     <xacro:standoff_rod rod_name="front_right_rod" origin_xyz="0 0 0.110"
             origin_rpy="0 0 0" r_l="0.220" r_r="0.01" material="white" mass="0.250"/>
-    <xacro:rod_joint joint_name="front_right_rod_joint" type="continuous"
-        origin_xyz="0.090 -0.090 0.1902" origin_rpy="0 0 0" parent="base_link"
+    <xacro:rod_joint joint_name="front_right_rod_joint" type="fixed"
+        origin_xyz="0.050 -0.130 0.1902" origin_rpy="0 0 0" parent="base_link"
         child="front_right_rod"/>
     <gazebo reference="front_right_rod">
@@ -146,6 +147,6 @@
     <xacro:standoff_rod rod_name="front_left_rod" origin_xyz="0 0 0.110"
             origin_rpy="0 0 0" r_l="0.220" r_r="0.01" material="white" mass="0.250"/>
-    <xacro:rod_joint joint_name="front_left_rod_joint" type="continuous"
-        origin_xyz="0.090 0.090 0.1902" origin_rpy="0 0 0" parent="base_link"
+    <xacro:rod_joint joint_name="front_left_rod_joint" type="fixed"
+        origin_xyz="0.050 0.130 0.1902" origin_rpy="0 0 0" parent="base_link"
         child="front_left_rod"/>
     <gazebo reference="front_left_rod">
@@ -155,6 +156,6 @@
     <xacro:standoff_rod rod_name="back_right_rod" origin_xyz="0 0 0.110"
             origin_rpy="0 0 0" r_l="0.220" r_r="0.01" material="white" mass="0.250"/>
-    <xacro:rod_joint joint_name="back_right_rod_joint" type="continuous"
-        origin_xyz="-0.090 -0.090 0.1902" origin_rpy="0 0 0" parent="base_link"
+    <xacro:rod_joint joint_name="back_right_rod_joint" type="fixed"
+        origin_xyz="-0.020 -0.130 0.1902" origin_rpy="0 0 0" parent="base_link"
         child="back_right_rod"/>
     <gazebo reference="back_right_rod">
@@ -164,6 +165,6 @@
     <xacro:standoff_rod rod_name="back_left_rod" origin_xyz="0 0 0.110"
             origin_rpy="0 0 0" r_l="0.220" r_r="0.01" material="white" mass="0.250"/>
-    <xacro:rod_joint joint_name="back_left_rod_joint" type="continuous"
-        origin_xyz="-0.090 0.090 0.1902" origin_rpy="0 0 0" parent="base_link"
+    <xacro:rod_joint joint_name="back_left_rod_joint" type="fixed"
+        origin_xyz="-0.020 0.130 0.1902" origin_rpy="0 0 0" parent="base_link"
         child="back_left_rod"/>
     <gazebo reference="back_left_rod">
@@ -173,5 +174,5 @@
     <xacro:cup_holder_tray link_name="cup_holder" origin_xyz="0 0 0"
             origin_rpy="0 0 0" cht_l="0.090" cht_r="0.160" material="blue" mass="1.0"/>
-    <xacro:cup_holder_tray_joint joint_name="cup_holder_joint" type="continuous"
+    <xacro:cup_holder_tray_joint joint_name="cup_holder_joint" type="fixed"
         origin_xyz="0 0 0.4552" origin_rpy="0 0 0" parent="base_link"
         child="cup_holder"/>
@@ -180,72 +181,4 @@
     </gazebo>
     <!--********************Laser Scan **************************-->
-    <xacro:macro name="laser" params="include_laser:=true">
-        <xacro:if value="${include_laser}">
-            <!-- Laser Sensor -->
-            <link name="laser_scan_link">
-                <visual>
-                    <origin rpy="0 0 0" xyz="0 0 -0.04"/>
-                    <geometry>
-                        <mesh filename="package://barista_robot_description/meshes/hokuyo_urg_04lx.dae" scale="1.0 1.0 1.0"/>
-                    </geometry>
-                </visual>
-                <collision>
-                    <origin rpy="0 0 0" xyz="0 0 0"/>
-                    <geometry>
-                        <box size="0.1 0.1 0.08"/>
-                    </geometry>
-                </collision>
-                <inertial>
-                    <mass value="0.160"/>
-                    <origin rpy="0 0 0" xyz="0 0 0"/>
-                    <inertia ixx="0.0002186666666666667" ixy="0" ixz="0" iyy="0.0002186666666666667" iyz="0" izz="0.00026666666666666673"/>
-                </inertial>
-            </link>
-            <joint name="laser_scan_link_joint" type="fixed">
-                <origin rpy="0 0 0" xyz="0.090 0 0.2302"/> <!--z = 0.0352 + 0.155 + 0.08/2-->
-                <parent link="base_link"/>
-                <child link="laser_scan_link"/>
-            </joint>
-            <gazebo reference="laser_scan_link">
-                <mu1>10.0</mu1>
-                <mu2>10.0</mu2>
-                <material>Gazebo/Grey</material>
-            </gazebo>
-            <gazebo reference="laser_scan_link">
-                <sensor name="sensor_ray" type="ray">
-                    <pose>0 0 0 0 0 0</pose>
-                    <ray>
-                        <scan>
-                            <horizontal>
-                                <samples>200</samples>
-                                <resolution>1.0</resolution>
-                                <min_angle>-1.5707</min_angle>
-                                <max_angle>1.5707</max_angle>
-                            </horizontal>
-                        </scan>
-                        <range>
-                            <min>0.2</min>
-                            <max>4.0</max>
-                        </range>
-                        <noise>
-                            <type>gaussian</type>
-                            <mean>0.0</mean>
-                            <stddev>0.01</stddev>
-                        </noise>
-                    </ray>
-                    <always_on>true</always_on>
-                    <visualize>true</visualize>
-                    <update_rate>100</update_rate>
-                    <plugin name="laser" filename="libgazebo_ros_ray_sensor.so">
-                        <ros>
-                            <!-- <namespace>/barista_robot</namespace> -->
-                            <remapping>~/out:=scan</remapping>
-                        </ros>
-                        <output_type>sensor_msgs/LaserScan</output_type>
-                    </plugin>
-                </sensor>
-            </gazebo>
-        </xacro:if>
-    </xacro:macro>
     <xacro:laser include_laser="${include_laser}"/>
     <!--********************Differential Drive Plugin **************************-->

Commit message: Adjusted files to spawn two instances of barista_bot

File: xacro/barista_robot_model.urdf.xacro (robot description, xacro)
@@ -12,4 +12,7 @@
     <xacro:property name="include_laser" value="true"/>
     <xacro:include filename="$(find barista_robot_description)/xacro/laser_scanner.xacro"/>
+    <!-- Add disfferent names and colors to spawn multiple robots -->
+    <xacro:property name="robot_name" value="$(arg robot_name)"/>
+    <xacro:property name="robot_gazebo_material" value="$(arg robot_gazebo_material)"/>
     <material name="red">
       <color rgba="1.0 0.0 0.0 1"/>
@@ -59,5 +62,5 @@
     </joint>
     <gazebo reference="chassis">
-        <material>Gazebo/Blue</material>
+        <material>${robot_gazebo_material}</material>
     </gazebo>
     <!--******************** Drive Wheels **************************-->
@@ -178,8 +181,26 @@
         child="cup_holder"/>
     <gazebo reference="cup_holder">
-        <material>Gazebo/Blue</material>
+        <material>${robot_gazebo_material}</material>
+    </gazebo>
+    <!-- ****************** Joint State Publisher *********************-->
+    <gazebo>
+        <plugin name="barista_bot_joint_state" filename="libgazebo_ros_joint_state_publisher.so">
+            <ros>
+                <namespace>/${robot_name}</namespace>
+                <remapping>~/out:=joint_states</remapping>
+            </ros>
+            <update_rate>30</update_rate>
+            <joint_name>right_motor_wheel_joint</joint_name>
+            <joint_name>left_motor_wheel_joint</joint_name>
+            <joint_name>front_yaw_joint</joint_name>
+            <joint_name>back_yaw_joint</joint_name>
+            <joint_name>front_roll_joint</joint_name>
+            <joint_name>back_roll_joint</joint_name>
+            <joint_name>front_pitch_joint</joint_name>
+            <joint_name>back_pitch_joint</joint_name>
+        </plugin>
     </gazebo>
     <!--********************Laser Scan **************************-->
-    <xacro:laser include_laser="${include_laser}"/>
+    <xacro:laser include_laser="${include_laser}" robot_name="${robot_name}"/>
     <!--********************Differential Drive Plugin **************************-->
     <gazebo>
@@ -195,10 +216,13 @@
             <max_wheel_acceleration>2.0</max_wheel_acceleration>
             <!-- Topic to receive geometry_msgs/Twist message commands, defaults to `cmd_vel` -->
-            <commandTopic>cmd_vel</commandTopic>
+            <ros>
+                <namespace>/${robot_name}</namespace>
+                <remapping>/cmd_vel:=cmd_vel</remapping>
+            </ros>
             <!-- output -->
             <publish_odom>true</publish_odom>
             <publish_odom_tf>true</publish_odom_tf>
-            <odometry_frame>odom</odometry_frame>
-            <robot_base_frame>base_link</robot_base_frame>
+            <odometry_frame>${robot_name}/odom</odometry_frame>
+            <robot_base_frame>${robot_name}/base_link</robot_base_frame>
         </plugin>
     </gazebo>

File: xacro/laser_scanner.xacro (robot description, xacro)
@@ -1,5 +1,5 @@
 <?xml version="1.0"?>
 <robot xmlns:xacro="http://www.ros.org/wiki/xacro">
-    <xacro:macro name="laser" params="include_laser:=true">
+    <xacro:macro name="laser" params="include_laser:=true robot_name">
         <xacro:if value="${include_laser}">
             <!-- Laser Sensor -->
@@ -46,5 +46,5 @@
                         <range>
                             <min>0.2</min>
-                            <max>30.0</max>
+                            <max>10.0</max>
                             <resolution>0.01</resolution>
                         </range>
@@ -57,4 +57,5 @@
                     <plugin name="laser_controller" filename="libgazebo_ros_ray_sensor.so">
                         <ros>
+                            <namespace>/${robot_name}</namespace>
                             <remapping>~/out:=scan</remapping>
                         </ros>

Commit message: Added new world tf to visualize both robots in RVIZ

File: xacro/barista_robot_model.urdf.xacro (robot description, xacro)
@@ -15,4 +15,5 @@
     <xacro:property name="robot_name" value="$(arg robot_name)"/>
     <xacro:property name="robot_gazebo_material" value="$(arg robot_gazebo_material)"/>
+    <xacro:property name="robot_rviz_material" value="$(arg robot_rviz_material)"/>
     <material name="red">
       <color rgba="1.0 0.0 0.0 1"/>
@@ -42,5 +43,5 @@
                     <cylinder length="0.155" radius="0.178"/>
                 </geometry>
-            <material name="blue"/>
+            <material name="${robot_rviz_material}"/>
         </visual>
         <collision>
@@ -176,5 +177,5 @@
     <!--******************** Cup Holder Tray **************************-->
     <xacro:cup_holder_tray link_name="cup_holder" origin_xyz="0 0 0"
-            origin_rpy="0 0 0" cht_l="0.090" cht_r="0.160" material="blue" mass="1.0"/>
+            origin_rpy="0 0 0" cht_l="0.090" cht_r="0.160" material="${robot_rviz_material}" mass="1.0"/>
     <xacro:cup_holder_tray_joint joint_name="cup_holder_joint" type="fixed"
         origin_xyz="0 0 0.4552" origin_rpy="0 0 0" parent="base_link"
